Commit message: Lowered to 70 deg ringpinkie to avoid self collision

File: src/lerobot/robots/ergocub/ergocub_hand_left/model.urdf (robot description, URDF)
Before this commit: robot ergocub_hand_left, 19 links, 18 joints
Joints:
- joint l_051ring1: limit lower=0 upper=1.57080 effort=4 velocity=4 -> lower=0 upper=1.2217 effort=4 velocity=4
- joint l_053pinkie1: limit lower=0 upper=1.57080 effort=4 velocity=4 -> lower=0 upper=1.2217 effort=4 velocity=4

File: src/lerobot/robots/ergocub/ergocub_hand_right/model.urdf (robot description, URDF)
Before this commit: robot ergocub_hand_right, 19 links, 18 joints
Joints:
- joint r_051ring1: limit lower=0 upper=1.5707963267948966 effort=4 velocity=4 -> lower=0 upper=1.2217 effort=4 velocity=4
- joint r_053pinkie1: limit lower=0 upper=1.5707963267948966 effort=4 velocity=4 -> lower=0 upper=1.2217 effort=4 velocity=4
